File: Kicad/Fluke 9010a Probe/Fluke 9010a Probe.kicad_pcb (KiCad board)
At the start: 2 copper layers, 58 x 8.2 mm, 19 parts, among them Q1 MMBT3906, Q2 MMBT3904

Commit message: latest
Parts:
- TP1: footprint Connector_PinSocket_2.54mm:PinSocket_1x01_P2.54mm_Vertical -> TestPoint:TestPoint_THTPad_3.0x3.0mm_Drill1.5mm
- moved C3 0.51 mm to (123.7, 123.8)
- moved R1 0.51 mm to (123.6, 123.8)
- turned C4 to 0 degrees
Routing:
- net /PULSELO: track 23.6 -> 26.2 mm, vias 2 -> 0
- net /-.7V: track 22.7 -> 25.2 mm
- net Net-(C1-Pad2): track 67.2 -> 65.8 mm
- net /~PULSEHI: track 13.7 -> 13.1 mm
Other:
- board text added: "v1.5"
- board text removed: "v1.3"
