File: Kicad/Fluke 9010a Probe/Fluke 9010a Probe.sch (KiCad schematic (older format))
At the start: 18 parts, among them Q1 MMBT3906, Q2 MMBT3904

Commit message: latest
Parts:
- TP1: footprint Connector_PinSocket_2.54mm:PinSocket_1x01_P2.54mm_Vertical -> TestPoint:TestPoint_THTPad_3.0x3.0mm_Drill1.5mm
Changed lines of the file:
@@
 Comment1 ""
 Comment2 ""
-Comment3 "M. Biry"
+Comment3 "Zubline"
 Comment4 ""
 $EndDescr
@@
 F 0 "TP1" H 9002 2601 50  0000 L CNN
 F 1 "Probe Tip" H 9250 2600 50  0000 L CNN
-F 2 "Connector_PinSocket_2.54mm:PinSocket_1x01_P2.54mm_Vertical" H 9050 2500 50  0001 C CNN
+F 2 "TestPoint:TestPoint_THTPad_3.0x3.0mm_Drill1.5mm" H 9050 2500 50  0001 C CNN
 F 3 "~" H 9050 2500 50  0001 C CNN
 	1    8850 2500
